File: KiCad files/Long range deauther.sch (KiCad schematic (older format))
At the start: 25 parts, among them J1 USB-AM-S-X-X-TH, Q1 BC847, Q2 BC847, SW1 SW_Flash, SW2 SW_RST, U1 NCP1117-3.3_SOT223, U2 CP2102N-A02-GQFN28, U3 ESP-WROOM-02U

Commit message: next update with some update on pcb
these updates are for use and for production.
Changes are quickly listed in the changes.txt
Parts:
- removed D1: SP0503BAHT, Package_TO_SOT_SMD:SOT-143, symbol Power_Protection:SP0503BAHT
- removed J1: USB-AM-S-X-X-TH, Deauth_usb:SAMTEC_USB-AM-S-X-X-TH, symbol Long-range-deauther-rescue:USB-AM-S-X-X-TH-Deauth_Usb_Symbol
- removed U1: NCP1117-3.3_SOT223, Package_TO_SOT_SMD:SOT-223-3_TabPin2, symbol Regulator_Linear:NCP1117-3.3_SOT223
- removed U2: CP2102N-A02-GQFN28, Deauth_usb:CP2102N-A02-GQFN28, symbol Long-range-deauther-rescue:CP2102N-A02-GQFN28-Deauth_Usb_Symbol
- added C3: 47pF, Capacitor_SMD:C_0805_2012Metric_Pad1.15x1.40mm_HandSolder, symbol Device:C
- added C4, C8: 100nF, Capacitor_SMD:C_0805_2012Metric_Pad1.15x1.40mm_HandSolder, symbol Device:C
- added C6: 4.7uF, Capacitor_SMD:C_0805_2012Metric_Pad1.15x1.40mm_HandSolder, symbol Device:C
- added FB1: Ferrite_Bead, Capacitor_SMD:C_0805_2012Metric_Pad1.15x1.40mm_HandSolder, symbol Device:Ferrite_Bead
- added J1: USB_A, Connector_USB:USB_A_CNCTech_1001-011-01101_Horizontal, symbol Connector:USB_A
- added U1: AP2112-3.3, Long_range_deauther:AP2112_REGULATOR, symbol Long-range-deauther-rescue:AP2112-3.3
- added U2: FT231XS, Package_SO:SSOP-20_3.9x8.7mm_P0.635mm, symbol Interface_USB:FT231XS
- C1: value 4.7uF -> 10nF
- C2: value 0.1uF -> 47pF
- C5: renamed from C3; value 4.7uF -> 10uF
- C7: renamed from C4; value 0.1uF -> 10uF
- R1: value 22.1K -> 10K
- R2: value 47.5K -> 27R
- R3: value 1K -> 27R
- SW1: renamed from SW2; footprint Button_Switch_SMD:SW_Push_SPST_NO_Alps_SKRK -> Long_range_deauther:HYP_1TS003B-1600-3500A-CT
- SW2: renamed from SW1; footprint Button_Switch_SMD:SW_Push_SPST_NO_Alps_SKRK -> Long_range_deauther:HYP_1TS003B-1600-3500A-CT
- U3: footprint Deauth_usb:ESP-WROOM-02U -> Long_range_deauther:ESP-WROOM-02U; symbol Long-range-deauther-rescue:ESP-WROOM-02U-Deauth_Usb_Symbol -> Long-range-deauther-rescue:ESP-WROOM-02U-Deauth_Usb_Symbol-Long-range-deauther-rescue
- renumbered R6 to R10, R12 to R11, R8 to R12, R11 to R6, R10 to R7, R7 to R8
Connections:
- net +3V3: now also U1.5 (OUT); no longer R3.1
- net +5V: now also C4.1, C6.1, FB1.1, U1.1 (IN), U2.15 (VCC); no longer C1.1, C2.1
- net CP_RST: now also U2.2 (~RTS)
- net D+: now also R2.1, U2.11 (USBDP)
- net D-: now also R3.2, U2.12 (USBDM)
- net DTR: now also U2.1 (~DTR)
- net GND: now also C2.1, C3.2, C4.2, C6.2, C8.2, J1.4 (GND), J1.5 (Shield), U1.2 (GND), U2.16 (GND), U2.6 (GND); no longer C2.2, R2.2
- net RXD: now also U2.4 (RXD)
- net TXD: now also U2.20 (TXD)
- net at R1.2: now also U1.3 (EN); no longer R2.1
- new net: C1.1, FB1.2, J1.1 (VBUS)
- new net FTDI_100nF_TG: C8.1, U2.13 (3V3OUT), U2.14 (~RESET), U2.3 (VCCIO)
- new net J_N: C2.2, J1.2 (D-), R3.1
- new net J_P: C3.1, J1.3 (D+), R2.2
- no-connect marks 23 -> 15
Other:
- note added: "Power filtering"
- moved on the sheet: C5, C7
