File: KiCad files/deauther-andromeda.sch (KiCad schematic (older format))
At the start: 31 parts, among them J1 USB_A, J2 Conn_01x03_Male, J3 Conn_01x03_Male, Q1 BC847, Q2 BC847, SW1 SW_RST, SW2 SW_Flash, U1 AP2112-3.3, U2 FT231XS, U3 ESP-WROOM-02U

Commit message: manufactoring update
Parts:
- U1: footprint Long_range_deauther:AP2112_REGULATOR -> deauther-andromeda:AP2112_REGULATOR
- U3: footprint Long_range_deauther:ESP-WROOM-02U -> deauther-andromeda:ESP-WROOM-02U
Changed lines of the file:
@@
 F 0 "U3" H 7250 4265 50  0000 C CNN
 F 1 "ESP-WROOM-02U" H 7250 4174 50  0000 C CNN
-F 2 "Long_range_deauther:ESP-WROOM-02U" H 7200 4050 50  0001 C CNN
+F 2 "deauther-andromeda:ESP-WROOM-02U" H 7200 4050 50  0001 C CNN
 F 3 "" H 7200 4050 50  0001 C CNN
 	1    7250 3600
@@
 F 0 "U1" H 1700 1365 50  0000 C CNN
 F 1 "AP2112-3.3" H 1700 1274 50  0000 C CNN
-F 2 "Long_range_deauther:AP2112_REGULATOR" H 1700 1100 50  0001 C CNN
+F 2 "deauther-andromeda:AP2112_REGULATOR" H 1700 1100 50  0001 C CNN
 F 3 "" H 1700 1100 50  0001 C CNN
 	1    1700 1100
