File: KiCad files/deauther-andromeda.kicad_pcb (KiCad board)
At the start: 2 copper layers, 43 x 16 mm, 35 parts, among them J1 USB_A, J2 Conn_01x03_Male, J3 Conn_01x03_Male, Q1 BC847, Q2 BC847, SW1 SW_RST, SW2 SW_Flash, U1 AP2112-3.3, U2 FT231XS, U3 ESP-WROOM-02U

Commit message: manufactoring update
Parts:
- U1: footprint Long_range_deauther:AP2112_REGULATOR -> deauther-andromeda:AP2112_REGULATOR
- U3: footprint Long_range_deauther:ESP-WROOM-02U -> deauther-andromeda:ESP-WROOM-02U
- moved U1 1.57 mm to (151.9, 77.5)
