File: Pannel/pannel_clean.kicad_pcb (KiCad board)
At the start: 2 copper layers, 86 x 90 mm, 354 parts, among them J1 USB_A, J2 Conn_01x03_Male, J3 Conn_01x03_Male, Q1 BC847, Q2 BC847, SW1 SW_RST, SW2 SW_Flash, U1 AP2112-3.3, U2 FT231XS, U3 ESP-WROOM-02U

Commit message: other production stuff
Parts:
- removed the REF** at (131.5, 122.0)
- removed the REF** at (88.5, 58.0)
- removed the REF** at (88.5, 122.0)
- removed the REF** at (131.5, 106.0)
- removed the REF** at (88.5, 106.0)
- removed the REF** at (131.5, 90.0)
- removed the REF** at (88.5, 90.0)
- removed the REF** at (131.5, 74.0)
- removed the REF** at (88.5, 74.0)
- removed the REF** at (131.5, 58.0)
- added C5: 10uF, Capacitor_SMD:C_0805_2012Metric_Pad1.15x1.40mm_HandSolder, B.Cu at (123.0, 115.4)
- added C5: 10uF, Capacitor_SMD:C_0805_2012Metric_Pad1.15x1.40mm_HandSolder, B.Cu at (80.0, 51.4)
- added C5: 10uF, Capacitor_SMD:C_0805_2012Metric_Pad1.15x1.40mm_HandSolder, B.Cu at (80.0, 115.4)
- added C5: 10uF, Capacitor_SMD:C_0805_2012Metric_Pad1.15x1.40mm_HandSolder, B.Cu at (123.0, 99.4)
- added C5: 10uF, Capacitor_SMD:C_0805_2012Metric_Pad1.15x1.40mm_HandSolder, B.Cu at (80.0, 99.4)
- added C5: 10uF, Capacitor_SMD:C_0805_2012Metric_Pad1.15x1.40mm_HandSolder, B.Cu at (123.0, 83.4)
- added C5: 10uF, Capacitor_SMD:C_0805_2012Metric_Pad1.15x1.40mm_HandSolder, B.Cu at (80.0, 83.4)
- added C5: 10uF, Capacitor_SMD:C_0805_2012Metric_Pad1.15x1.40mm_HandSolder, B.Cu at (123.0, 67.4)
- added C5: 10uF, Capacitor_SMD:C_0805_2012Metric_Pad1.15x1.40mm_HandSolder, B.Cu at (80.0, 67.4)
- added C5: 10uF, Capacitor_SMD:C_0805_2012Metric_Pad1.15x1.40mm_HandSolder, B.Cu at (123.0, 51.4)
- FID3: moved to B.Cu
- REF** (x10): renamed from C5; value 10uF -> SMA_Horizontal; footprint Capacitor_SMD:C_0805_2012Metric_Pad1.15x1.40mm_HandSolder -> Long_range_deauther:SMA_Horizontal; moved to F.Cu
- moved REF** 10.8 mm to (131.5, 122.0), turned to 270 degrees
- moved REF** 10.8 mm to (88.5, 122.0), turned to 270 degrees
- moved REF** 10.8 mm to (131.5, 106.0), turned to 270 degrees
- moved REF** 10.8 mm to (88.5, 106.0), turned to 270 degrees
- moved REF** 10.8 mm to (131.5, 90.0), turned to 270 degrees
- moved REF** 10.8 mm to (88.5, 90.0), turned to 270 degrees
- moved REF** 10.8 mm to (131.5, 74.0), turned to 270 degrees
- moved REF** 10.8 mm to (88.5, 74.0), turned to 270 degrees
- moved REF** 10.8 mm to (88.5, 58.0), turned to 270 degrees
- moved REF** 10.8 mm to (131.5, 58.0), turned to 270 degrees
Connections:
- REF** pad 2: Board_10-GND -> (no net)
- REF** pad 2: Board_1-GND -> (no net)
- REF** pad 2: Board_9-GND -> (no net)
- REF** pad 2: Board_8-GND -> (no net)
- REF** pad 2: Board_7-GND -> (no net)
- REF** pad 2: Board_6-GND -> (no net)
- REF** pad 2: Board_5-GND -> (no net)
- REF** pad 2: Board_4-GND -> (no net)
- REF** pad 2: Board_3-GND -> (no net)
- REF** pad 2: Board_2-GND -> (no net)
